Commit message: Control&Gazebo: Gazebo > Propeller x-position adjusted

File: gazebo/urdf/drone.urdf (robot description, URDF)
Before this commit: robot custom_drone, 10 links, 9 joints
Joints:
- joint arm1_propeller1: origin xyz=0.1905255888325765 0.08999999999999998 0.015 rpy=0 0 0 -> xyz=0.15588457268119896 0.08999999999999998 0.015 rpy=0 0 0
- joint arm3_propeller3: origin xyz=-0.19052558883257648 0.09000000000000005 0.015 rpy=0 0 0 -> xyz=-0.15588457268119893 0.09000000000000005 0.015 rpy=0 0 0
- joint arm4_propeller4: origin xyz=-0.19052558883257653 -0.08999999999999994 0.015 rpy=0 0 0 -> xyz=-0.15588457268119899 -0.08999999999999994 0.015 rpy=0 0 0
- joint arm6_propeller6: origin xyz=0.19052558883257653 -0.08999999999999994 0.015 rpy=0 0 0 -> xyz=0.15588457268119899 -0.08999999999999994 0.015 rpy=0 0 0

File: gazebo/urdf/drone.xacro (robot description, xacro)
@@ -144,5 +144,5 @@
       <parent link="arm${i}"/>
       <child link="propeller${i}"/>
-      <origin xyz="${cos((i-1)*pi/3+pi/6)*(frame_radius+0.12)} ${sin((i-1)*pi/3+pi/6)*(0.08+arm_length_y)} ${0.04/2-arm_radius}" rpy="0 0 0"/>
+      <origin xyz="${cos((i-1)*pi/3+pi/6)*(frame_radius+0.08)} ${sin((i-1)*pi/3+pi/6)*(0.08+arm_length_y)} ${0.04/2-arm_radius}" rpy="0 0 0"/>
       <axis xyz="0 0 1"/>
       <limit lower="0" upper="0" effort="0" velocity="0"/>

Commit message: Control&Gazebo: Added gazebo_ros_control as controller for drone model

File: gazebo/urdf/drone.urdf (robot description, URDF)
Before this commit: robot custom_drone, 10 links, 9 joints
Links:
- link propeller1: geometry collision box size=0.011006666666666666 0.16000000000000003 0.001; visual box size=0.011006666666666666 0.16000000000000003 0.001
- link propeller3: geometry collision box size=0.011006666666666666 0.16000000000000003 0.001; visual box size=0.011006666666666666 0.16000000000000003 0.001
- link propeller4: geometry collision box size=0.011006666666666666 0.16000000000000003 0.001; visual box size=0.011006666666666666 0.16000000000000003 0.001
- link propeller6: geometry collision box size=0.011006666666666666 0.16000000000000003 0.001; visual box size=0.011006666666666666 0.16000000000000003 0.001
Joints:
- joint arm1_propeller1: limit lower=0 upper=0 effort=0 velocity=0 -> lower=-2.0 upper=2.0 effort=1000 velocity=3.0
- joint arm3_propeller3: limit lower=0 upper=0 effort=0 velocity=0 -> lower=-2.0 upper=2.0 effort=1000 velocity=3.0
- joint arm4_propeller4: limit lower=0 upper=0 effort=0 velocity=0 -> lower=-2.0 upper=2.0 effort=1000 velocity=3.0
- joint arm6_propeller6: limit lower=0 upper=0 effort=0 velocity=0 -> lower=-2.0 upper=2.0 effort=1000 velocity=3.0

File: gazebo/urdf/drone.xacro (robot description, xacro)
@@ -127,5 +127,6 @@
         <origin xyz="0 0 0" rpy="0 0 0"/>
         <geometry>
-          <cylinder radius="${propeller_radius_smaller}" length="${propeller_height}"/>
+          <!-- <cylinder radius="${propeller_radius_smaller}" length="${propeller_height}"/> -->
+          <box size="${0.03302/3} ${0.20*0.8} ${0.001}" />
         </geometry>
         <material name="propeller_material"/>
@@ -134,5 +135,6 @@
         <origin xyz="0 0 0" rpy="0 0 0"/>
         <geometry>
-          <cylinder radius="${propeller_radius_smaller}" length="${propeller_height}"/>
+          <!-- <cylinder radius="${propeller_radius_smaller}" length="${propeller_height}"/> -->
+          <box size="${0.03302/3} ${0.20*0.8} ${0.001}" />
         </geometry>
       </collision>
@@ -146,6 +148,16 @@
       <origin xyz="${cos((i-1)*pi/3+pi/6)*(frame_radius+0.08)} ${sin((i-1)*pi/3+pi/6)*(0.08+arm_length_y)} ${0.04/2-arm_radius}" rpy="0 0 0"/>
       <axis xyz="0 0 1"/>
-      <limit lower="0" upper="0" effort="0" velocity="0"/>
-    </joint>
+      <limit lower="-2.0" upper="2.0" effort="1000" velocity="3.0"/>
+    </joint>
+    <!-- <transmission name="transmission_propeller${i}">
+      <type>transmission_interface/SimpleTransmission</type>
+      <joint name="arm${i}_propeller${i}">
+        <hardwareInterface>EffortJointInterface</hardwareInterface>
+      </joint>
+      <actuator name="propeller${i}_motor">
+        <hardwareInterface>EffortJointInterface</hardwareInterface>
+        <mechanicalReduction>1</mechanicalReduction>
+      </actuator>
+    </transmission> -->
   </xacro:macro>
   <xacro:macro name="arm" params="i">
@@ -197,11 +209,161 @@
   <xacro:propeller i="4"/>
   <xacro:propeller i="6"/>
+  <!-- Transmissions -->
+  <transmission name="transmission_propeller1">
+    <type>transmission_interface/SimpleTransmission</type>
+    <joint name="arm1_propeller1">
+      <hardwareInterface>EffortJointInterface</hardwareInterface>
+    </joint>
+    <actuator name="propeller1_motor">
+      <hardwareInterface>EffortJointInterface</hardwareInterface>
+      <mechanicalReduction>1</mechanicalReduction>
+    </actuator>
+  </transmission>
+  <transmission name="transmission_propeller1">
+    <type>transmission_interface/SimpleTransmission</type>
+    <joint name="arm1_propeller1">
+      <hardwareInterface>EffortJointInterface</hardwareInterface>
+    </joint>
+    <actuator name="propeller1_motor">
+      <hardwareInterface>EffortJointInterface</hardwareInterface>
+      <mechanicalReduction>1</mechanicalReduction>
+    </actuator>
+  </transmission>
+  <transmission name="transmission_propeller3">
+    <type>transmission_interface/SimpleTransmission</type>
+    <joint name="arm3_propeller3">
+      <hardwareInterface>EffortJointInterface</hardwareInterface>
+    </joint>
+    <actuator name="propeller3_motor">
+      <hardwareInterface>EffortJointInterface</hardwareInterface>
+      <mechanicalReduction>1</mechanicalReduction>
+    </actuator>
+  </transmission>
+  <transmission name="transmission_propeller4">
+    <type>transmission_interface/SimpleTransmission</type>
+    <joint name="arm4_propeller4">
+      <hardwareInterface>EffortJointInterface</hardwareInterface>
+    </joint>
+    <actuator name="propeller4_motor">
+      <hardwareInterface>EffortJointInterface</hardwareInterface>
+      <mechanicalReduction>1</mechanicalReduction>
+    </actuator>
+  </transmission>
+  <transmission name="transmission_propeller6">
+    <type>transmission_interface/SimpleTransmission</type>
+    <joint name="arm6_propeller6">
+      <hardwareInterface>EffortJointInterface</hardwareInterface>
+    </joint>
+    <actuator name="propeller6_motor">
+      <hardwareInterface>EffortJointInterface</hardwareInterface>
+      <mechanicalReduction>1</mechanicalReduction>
+    </actuator>
+  </transmission>
   <!-- Tello plugin for Gazebo -->
   <gazebo>
-      <plugin name="ControlPlugin" filename="libcontrol_plugin.so">
+      <!-- <gazebo>
+        <plugin name="gazebo_ros_control" filename="libgazebo_ros_control.so">
+          <robotNamespace>gazebo</robotNamespace>
+          <robotSimType>gazebo_ros_control/DefaultRobotHWSim</robotSimType>
+        </plugin>
+      </gazebo> -->
+      <!-- <plugin name="ControlPlugin" filename="libcontrol_plugin.so">
           <parameter name="use_sim_time" type="bool">1</parameter>
           <link_name>body</link_name>
           <center_of_mass>0 0 0</center_of_mass>
       </plugin>
+      <plugin name="BatteryPlugin" filename="libbattery_plugin.so">
+          <parameter name="use_sim_time" type="bool">1</parameter>
+          <link_name>body</link_name>
+          <center_of_mass>0 0 0</center_of_mass>
+      </plugin> -->
+      <plugin name="gazebo_ros_control" filename="libgazebo_ros_control.so">
+        <robotNamespace>gazebo</robotNamespace>
+        <controlPeriod>0.002</controlPeriod>
+        <robotSimType>gazebo_ros_control/DefaultRobotHWSim</robotSimType>
+        <legacyModeNS>true</legacyModeNS>
+        <alwaysOn>true</alwaysOn>
+        <updateRate>1000.0</updateRate>
+        <joint name="arm${1}_propeller${1}">
+          <pid>
+            <p>1000.0</p>
+            <i>0.01</i>
+            <d>0.01</d>
+            <iMax>1000.0</iMax>
+            <iMin>-1000.0</iMin>
+            <cmdMax>1000.0</cmdMax>
+            <cmdMin>-1000.0</cmdMin>
+          </pid>
+        </joint>
+        <joint name="arm${3}_propeller${3}">
+          <pid>
+            <p>1000.0</p>
+            <i>0.01</i>
+            <d>0.01</d>
+            <iMax>1000.0</iMax>
+            <iMin>-1000.0</iMin>
+            <cmdMax>1000.0</cmdMax>
+            <cmdMin>-1000.0</cmdMin>
+          </pid>
+        </joint>
+        <joint name="arm${4}_propeller${4}">
+          <pid>
+            <p>1000.0</p>
+            <i>0.01</i>
+            <d>0.01</d>
+            <iMax>1000.0</iMax>
+            <iMin>-1000.0</iMin>
+            <cmdMax>1000.0</cmdMax>
+            <cmdMin>-1000.0</cmdMin>
+          </pid>
+        </joint>
+        <joint name="arm${6}_propeller${6}">
+          <pid>
+            <p>1000.0</p>
+            <i>0.01</i>
+            <d>0.01</d>
+            <iMax>1000.0</iMax>
+            <iMin>-1000.0</iMin>
+            <cmdMax>1000.0</cmdMax>
+            <cmdMin>-1000.0</cmdMin>
+          </pid>
+        </joint>
+      </plugin>
+  </gazebo>
+  <gazebo reference="camera_link">
+    <sensor type="camera" name="camera1">
+      <update_rate>30.0</update_rate>
+      <camera name="head">
+        <horizontal_fov>1.3962634</horizontal_fov>
+        <image>
+          <width>800</width>
+          <height>800</height>
+          <format>R8G8B8</format>
+        </image>
+        <clip>
+          <near>0.02</near>
+          <far>300</far>
+        </clip>
+        <noise>
+          <type>gaussian</type>
+          <mean>0.0</mean>
+          <stddev>0.007</stddev>
+        </noise>
+      </camera>
+      <plugin name="camera_controller" filename="libgazebo_ros_camera.so">
+        <alwaysOn>true</alwaysOn>
+        <updateRate>0.0</updateRate>
+        <cameraName>gazebo/camera1</cameraName>
+        <imageTopicName>image_raw</imageTopicName>
+        <cameraInfoTopicName>camera_info</cameraInfoTopicName>
+        <frameName>camera_link</frameName>
+        <hackBaseline>0.07</hackBaseline>
+        <distortionK1>0.0</distortionK1>
+        <distortionK2>0.0</distortionK2>
+        <distortionK3>0.0</distortionK3>
+        <distortionT1>0.0</distortionT1>
+        <distortionT2>0.0</distortionT2>
+      </plugin>
+    </sensor>
   </gazebo>
 </robot>

Commit message: Control&Gazebo: Modified yaml file and model in xacro file

File: gazebo/urdf/drone.urdf (robot description, URDF)
Before this commit: robot custom_drone, 10 links, 9 joints
Links:
- added link dummy
- link body: mass 0.1 -> 0.88
Joints:
- added joint dummy_joint: type fixed, parent dummy, child body
- joint arm1_propeller1: limit lower=-2.0 upper=2.0 effort=1000 velocity=3.0 -> lower=-6.2830 upper=6.283 effort=0 velocity=0.0; origin xyz=0.15588457268119896 0.08999999999999998 0.015 rpy=0 0 0 -> xyz=0.15588457268119896 0.08999999999999998 0.016 rpy=0 0 0
- joint arm3_propeller3: limit lower=-2.0 upper=2.0 effort=1000 velocity=3.0 -> lower=-6.2830 upper=6.283 effort=0 velocity=0.0; origin xyz=-0.15588457268119893 0.09000000000000005 0.015 rpy=0 0 0 -> xyz=-0.15588457268119893 0.09000000000000005 0.016 rpy=0 0 0
- joint arm4_propeller4: limit lower=-2.0 upper=2.0 effort=1000 velocity=3.0 -> lower=-6.2830 upper=6.283 effort=0 velocity=0.0; origin xyz=-0.15588457268119899 -0.08999999999999994 0.015 rpy=0 0 0 -> xyz=-0.15588457268119899 -0.08999999999999994 0.016 rpy=0 0 0
- joint arm6_propeller6: limit lower=-2.0 upper=2.0 effort=1000 velocity=3.0 -> lower=-6.2830 upper=6.283 effort=0 velocity=0.0; origin xyz=0.15588457268119899 -0.08999999999999994 0.015 rpy=0 0 0 -> xyz=0.15588457268119899 -0.08999999999999994 0.016 rpy=0 0 0

File: gazebo/urdf/drone.xacro (robot description, xacro)
@@ -34,4 +34,6 @@
   <xacro:property name="arm_length_y" value="0.10"/>
   <xacro:property name="body_height" value="0.02"/>
+  <link name="dummy">
+   </link>
   <!-- Body link -->
   <link name="body">
@@ -50,34 +52,6 @@
           <material name="white"/>
       </visual>
-      <!-- <visual>
-          <origin xyz="0.05 -0.05 0"/>
-          <geometry>
-              <cylinder length="0.01" radius="0.045"/>
-          </geometry>
-          <material name="Gazebo/black"/>
-      </visual>
-      <visual>
-          <origin xyz="-0.05 0.05 0"/>
-          <geometry>
-              <cylinder length="0.01" radius="0.045"/>
-          </geometry>
-          <material name="black"/>
-      </visual>
-      <visual>
-          <origin xyz="-0.05 -0.05 0"/>
-          <geometry>
-              <cylinder length="0.01" radius="0.045"/>
-          </geometry>
-          <material name="black"/>
-      </visual>
-      <visual>
-          <origin xyz="0.05 0.05 0"/>
-          <geometry>
-              <cylinder length="0.01" radius="0.045"/>
-          </geometry>
-          <material name="black"/>
-      </visual> -->
       <inertial>
-          <mass value="0.1"/>
+          <mass value="${frame_mass}"/>
           <inertia ixx="0.000290833" ixy="0" ixz="0" iyy="0.00054" iyz="0" izz="0.000290833"/>
       </inertial>
@@ -88,4 +62,8 @@
       </collision>
   </link>
+  <joint name="dummy_joint" type="fixed">
+     <parent link="dummy"/>
+     <child link="body"/>
+  </joint>
   <!-- Camera link -->
   <link name="camera_link">
@@ -127,13 +105,11 @@
         <origin xyz="0 0 0" rpy="0 0 0"/>
         <geometry>
-          <!-- <cylinder radius="${propeller_radius_smaller}" length="${propeller_height}"/> -->
           <box size="${0.03302/3} ${0.20*0.8} ${0.001}" />
         </geometry>
-        <material name="propeller_material"/>
+        <material name="red"/>
       </visual>
       <collision>
         <origin xyz="0 0 0" rpy="0 0 0"/>
         <geometry>
-          <!-- <cylinder radius="${propeller_radius_smaller}" length="${propeller_height}"/> -->
           <box size="${0.03302/3} ${0.20*0.8} ${0.001}" />
         </geometry>
@@ -146,23 +122,13 @@
       <parent link="arm${i}"/>
       <child link="propeller${i}"/>
-      <origin xyz="${cos((i-1)*pi/3+pi/6)*(frame_radius+0.08)} ${sin((i-1)*pi/3+pi/6)*(0.08+arm_length_y)} ${0.04/2-arm_radius}" rpy="0 0 0"/>
+      <origin xyz="${cos((i-1)*pi/3+pi/6)*(frame_radius+0.08)} ${sin((i-1)*pi/3+pi/6)*(0.08+arm_length_y)} ${0.042/2-arm_radius}" rpy="0 0 0"/>
       <axis xyz="0 0 1"/>
-      <limit lower="-2.0" upper="2.0" effort="1000" velocity="3.0"/>
-    </joint>
-    <!-- <transmission name="transmission_propeller${i}">
-      <type>transmission_interface/SimpleTransmission</type>
-      <joint name="arm${i}_propeller${i}">
-        <hardwareInterface>EffortJointInterface</hardwareInterface>
-      </joint>
-      <actuator name="propeller${i}_motor">
-        <hardwareInterface>EffortJointInterface</hardwareInterface>
-        <mechanicalReduction>1</mechanicalReduction>
-      </actuator>
-    </transmission> -->
+      <limit lower="-6.2830" upper="6.283" effort="0" velocity="0.0"/>
+    </joint>
   </xacro:macro>
   <xacro:macro name="arm" params="i">
     <link name="arm${i}">
       <visual>
-        <origin xyz="${cos((i-1)*pi/3+pi/6)*(frame_radius+0.10/8)} ${sin((i-1)*pi/3+pi/6)*(0.05+arm_length_y/2)} ${body_height/2-arm_radius}" rpy="0 ${pi/2} ${(i-1)*pi/3+pi/6}"/>
+        <origin xyz="${cos((i-1)*pi/3+pi/6)*(frame_radius+0.10/8)} ${sin((i-1)*pi/3+pi/6)*(0.05+arm_length_y/2)} ${body_height/2-arm_radius}" rpy="0 ${pi/180 * 85} ${(i-1)*pi/3+pi/6}"/>
         <geometry>
           <cylinder radius="${arm_radius}" length="${arm_length}"/>
@@ -171,5 +137,5 @@
       </visual>
       <collision>
-        <origin xyz="${cos((i-1)*pi/3+pi/6)*(frame_radius+0.10/8)} ${sin((i-1)*pi/3+pi/6)*(0.05+arm_length_y/2)} ${body_height/2-arm_radius}" rpy="0 ${pi/2} ${(i-1)*pi/3+pi/6}"/>
+        <origin xyz="${cos((i-1)*pi/3+pi/6)*(frame_radius+0.10/8)} ${sin((i-1)*pi/3+pi/6)*(0.05+arm_length_y/2)} ${body_height/2-arm_radius}" rpy="0 ${pi/180 * 85} ${(i-1)*pi/3+pi/6}"/>
         <geometry>
           <cylinder radius="${arm_radius}" length="${arm_length}"/>
@@ -177,5 +143,5 @@
       </collision>
       <xacro:cylinder_inertial radius="${arm_radius}" height="${arm_length}" mass="${arm_mass}">
-        <origin xyz="${cos((i-1)*pi/3+pi/6)*(frame_radius+0.10/8)} ${sin((i-1)*pi/3+pi/6)*(0.05+arm_length_y/2)} ${body_height/2-arm_radius}" rpy="0 ${pi/2} ${(i-1)*pi/3+pi/6}"/>
+        <origin xyz="${cos((i-1)*pi/3+pi/6)*(frame_radius+0.10/8)} ${sin((i-1)*pi/3+pi/6)*(0.05+arm_length_y/2)} ${body_height/2-arm_radius}" rpy="0 $${pi/180 * 85} ${(i-1)*pi/3+pi/6}"/>
       </xacro:cylinder_inertial>
     </link>
@@ -202,6 +168,4 @@
   <xacro:arm i="3"/>
   <xacro:arm i="4"/>
-  <!-- <xacro:arm i="2"/> -->
-  <!-- <xacro:arm i="5"/> -->
   <xacro:arm i="6"/>
   <xacro:propeller i="1"/>
@@ -213,18 +177,8 @@
     <type>transmission_interface/SimpleTransmission</type>
     <joint name="arm1_propeller1">
-      <hardwareInterface>EffortJointInterface</hardwareInterface>
+      <hardwareInterface>hardware_interface/VelocityJointInterface</hardwareInterface>
     </joint>
     <actuator name="propeller1_motor">
-      <hardwareInterface>EffortJointInterface</hardwareInterface>
-      <mechanicalReduction>1</mechanicalReduction>
-    </actuator>
-  </transmission>
-  <transmission name="transmission_propeller1">
-    <type>transmission_interface/SimpleTransmission</type>
-    <joint name="arm1_propeller1">
-      <hardwareInterface>EffortJointInterface</hardwareInterface>
-    </joint>
-    <actuator name="propeller1_motor">
-      <hardwareInterface>EffortJointInterface</hardwareInterface>
+      <hardwareInterface>hardware_interface/VelocityJointInterface</hardwareInterface>
       <mechanicalReduction>1</mechanicalReduction>
     </actuator>
@@ -233,8 +187,8 @@
     <type>transmission_interface/SimpleTransmission</type>
     <joint name="arm3_propeller3">
-      <hardwareInterface>EffortJointInterface</hardwareInterface>
+      <hardwareInterface>hardware_interface/VelocityJointInterface</hardwareInterface>
     </joint>
     <actuator name="propeller3_motor">
-      <hardwareInterface>EffortJointInterface</hardwareInterface>
+      <hardwareInterface>hardware_interface/VelocityJointInterface</hardwareInterface>
       <mechanicalReduction>1</mechanicalReduction>
     </actuator>
@@ -243,8 +197,8 @@
     <type>transmission_interface/SimpleTransmission</type>
     <joint name="arm4_propeller4">
-      <hardwareInterface>EffortJointInterface</hardwareInterface>
+      <hardwareInterface>hardware_interface/VelocityJointInterface</hardwareInterface>
     </joint>
     <actuator name="propeller4_motor">
-      <hardwareInterface>EffortJointInterface</hardwareInterface>
+      <hardwareInterface>hardware_interface/VelocityJointInterface</hardwareInterface>
       <mechanicalReduction>1</mechanicalReduction>
     </actuator>
@@ -253,8 +207,8 @@
     <type>transmission_interface/SimpleTransmission</type>
     <joint name="arm6_propeller6">
-      <hardwareInterface>EffortJointInterface</hardwareInterface>
+      <hardwareInterface>hardware_interface/VelocityJointInterface</hardwareInterface>
     </joint>
     <actuator name="propeller6_motor">
-      <hardwareInterface>EffortJointInterface</hardwareInterface>
+      <hardwareInterface>hardware_interface/VelocityJointInterface</hardwareInterface>
       <mechanicalReduction>1</mechanicalReduction>
     </actuator>
@@ -262,72 +216,17 @@
   <!-- Tello plugin for Gazebo -->
   <gazebo>
-      <!-- <gazebo>
-        <plugin name="gazebo_ros_control" filename="libgazebo_ros_control.so">
-          <robotNamespace>gazebo</robotNamespace>
-          <robotSimType>gazebo_ros_control/DefaultRobotHWSim</robotSimType>
-        </plugin>
-      </gazebo> -->
-      <!-- <plugin name="ControlPlugin" filename="libcontrol_plugin.so">
-          <parameter name="use_sim_time" type="bool">1</parameter>
-          <link_name>body</link_name>
-          <center_of_mass>0 0 0</center_of_mass>
+      <plugin name="gazebo_ros_control" filename="libgazebo_ros_control.so">
+        <robotNamespace>/control</robotNamespace>
       </plugin>
-      <plugin name="BatteryPlugin" filename="libbattery_plugin.so">
-          <parameter name="use_sim_time" type="bool">1</parameter>
-          <link_name>body</link_name>
-          <center_of_mass>0 0 0</center_of_mass>
-      </plugin> -->
-      <plugin name="gazebo_ros_control" filename="libgazebo_ros_control.so">
-        <robotNamespace>gazebo</robotNamespace>
-        <controlPeriod>0.002</controlPeriod>
-        <robotSimType>gazebo_ros_control/DefaultRobotHWSim</robotSimType>
-        <legacyModeNS>true</legacyModeNS>
-        <alwaysOn>true</alwaysOn>
-        <updateRate>1000.0</updateRate>
-        <joint name="arm${1}_propeller${1}">
-          <pid>
-            <p>1000.0</p>
-            <i>0.01</i>
-            <d>0.01</d>
-            <iMax>1000.0</iMax>
-            <iMin>-1000.0</iMin>
-            <cmdMax>1000.0</cmdMax>
-            <cmdMin>-1000.0</cmdMin>
-          </pid>
-        </joint>
-        <joint name="arm${3}_propeller${3}">
-          <pid>
-            <p>1000.0</p>
-            <i>0.01</i>
-            <d>0.01</d>
-            <iMax>1000.0</iMax>
-            <iMin>-1000.0</iMin>
-            <cmdMax>1000.0</cmdMax>
-            <cmdMin>-1000.0</cmdMin>
-          </pid>
-        </joint>
-        <joint name="arm${4}_propeller${4}">
-          <pid>
-            <p>1000.0</p>
-            <i>0.01</i>
-            <d>0.01</d>
-            <iMax>1000.0</iMax>
-            <iMin>-1000.0</iMin>
-            <cmdMax>1000.0</cmdMax>
-            <cmdMin>-1000.0</cmdMin>
-          </pid>
-        </joint>
-        <joint name="arm${6}_propeller${6}">
-          <pid>
-            <p>1000.0</p>
-            <i>0.01</i>
-            <d>0.01</d>
-            <iMax>1000.0</iMax>
-            <iMin>-1000.0</iMin>
-            <cmdMax>1000.0</cmdMax>
-            <cmdMin>-1000.0</cmdMin>
-          </pid>
-        </joint>
-      </plugin>
+  </gazebo>
+  <gazebo>
+    <plugin name="gazebo_ros_joint_state_publisher"
+        filename="libgazebo_ros_joint_state_publisher.so">
+        <update_rate>20</update_rate>
+        <joint_name>arm1_propeller1</joint_name>
+        <joint_name>arm3_propeller3</joint_name>
+        <joint_name>arm4_propeller4</joint_name>
+        <joint_name>arm6_propeller6</joint_name>
+    </plugin>
   </gazebo>
   <gazebo reference="camera_link">
