Commit message: Control&Gazebo: Added command classes, action and service files

File: gazebo/urdf/drone.urdf (robot description, URDF)
Before this commit: robot custom_drone, 11 links, 10 joints
Joints:
- joint arm1_propeller1: limit lower=-6.2830 upper=6.283 effort=0 velocity=0.0 -> lower=-6.2830 upper=6.283 effort=2 velocity=2.0
- joint arm3_propeller3: limit lower=-6.2830 upper=6.283 effort=0 velocity=0.0 -> lower=-6.2830 upper=6.283 effort=2 velocity=2.0
- joint arm4_propeller4: limit lower=-6.2830 upper=6.283 effort=0 velocity=0.0 -> lower=-6.2830 upper=6.283 effort=2 velocity=2.0
- joint arm6_propeller6: limit lower=-6.2830 upper=6.283 effort=0 velocity=0.0 -> lower=-6.2830 upper=6.283 effort=2 velocity=2.0

File: gazebo/urdf/drone.xacro (robot description, xacro)
@@ -124,5 +124,5 @@
       <origin xyz="${cos((i-1)*pi/3+pi/6)*(frame_radius+0.08)} ${sin((i-1)*pi/3+pi/6)*(0.08+arm_length_y)} ${0.042/2-arm_radius}" rpy="0 0 0"/>
       <axis xyz="0 0 1"/>
-      <limit lower="-6.2830" upper="6.283" effort="0" velocity="0.0"/>
+      <limit lower="-6.2830" upper="6.283" effort="2" velocity="2.0"/>
     </joint>
   </xacro:macro>
